File: shematic/sheematic/processor.sch (KiCad schematic (older format))
At the start: 1 part

Commit message: cpu updated
Parts:
- removed U?: STM32F103C4Tx, Package_QFP:LQFP-48_7x7mm_P0.5mm, symbol MCU_ST_STM32F1:STM32F103C4Tx
- added C? (x4): C, symbol Device:C
- added J? (x3): Conn_01x05_Male, symbol Connector:Conn_01x05_Male
- added J?: Conn_01x02_Male, symbol Connector:Conn_01x02_Male
- added J? (x4): Conn_01x07_Male, symbol Connector:Conn_01x07_Male
- added L?: L, symbol Device:L
- added U1: E73-2G4M04S-52832, RF_Module:E73-2G4M04S, symbol RF_Module:E73-2G4M04S-52832
Connections:
- net labels added: +3.3V, GND, SCL, SDA
- wire segments 0 -> 90

Commit message: updated
Parts:
- added J?: LCD, symbol Connector:Conn_01x08_Male
- gave numbers to parts that had none: 13
Connections:
- net +3V3: now also J?.2 (Pin_2), J?.8 (Pin_8)
- net GND: now also J?.1 (Pin_1)
- net CCS811_nINT: now reaches J6.1 (Pin_1), U1.26 (P0.11)
- net CCS811_nRESET: now reaches J6.2 (Pin_2), U1.27 (P0.12)
- net CCS811_nWAKE: now reaches J6.3 (Pin_3), U1.28 (P0.13)
- net dis_SCK: now reaches J6.4 (Pin_4), U1.29 (P0.14)
- net dis_SCK: now also J?.3 (Pin_3)
- net dis_SDA: now reaches J6.5 (Pin_5), U1.30 (P0.15)
- net dis_SDA: now also J?.4 (Pin_4)
- net dis_RES: now reaches J6.6 (Pin_6), U1.31 (P0.16)
- net dis_RES: now also J?.5 (Pin_5)
- net dis_RS: now reaches J6.7 (Pin_7), U1.32 (P0.17)
- net dis_RS: now also J?.6 (Pin_6)
- net dis_CS: now reaches J7.1 (Pin_1), U1.33 (SWO/P0.18)
- net dis_CS: now also J?.7 (Pin_7)
Changed lines of the file:
@@
 $EndComp
 $Comp
-L power:GND #PWR?
+L power:GND #PWR06
 U 1 1 602A52CE
 P 6150 4650
-F 0 "#PWR?" H 6150 4400 50  0001 C CNN
+F 0 "#PWR06" H 6150 4400 50  0001 C CNN
 F 1 "GND" H 6155 4477 50  0000 C CNN
 F 2 "" H 6150 4650 50  0001 C CNN
@@
 	6150 4650 6150 4500
 $Comp
-L Connector:Conn_01x05_Male J?
+L Connector:Conn_01x05_Male J3
 U 1 1 602A64EC
 P 4700 3600
-F 0 "J?" H 4808 3981 50  0000 C CNN
+F 0 "J3" H 4808 3981 50  0000 C CNN
 F 1 "Conn_01x05_Male" H 4808 3890 50  0000 C CNN
 F 2 "" H 4700 3600 50  0001 C CNN
@@
 Connection ~ 6150 4500
 $Comp
-L power:+3.3V #PWR?
+L power:+3.3V #PWR05
 U 1 1 602A7D4A
 P 6150 1100
-F 0 "#PWR?" H 6150 950 50  0001 C CNN
+F 0 "#PWR05" H 6150 950 50  0001 C CNN
 F 1 "+3.3V" H 6165 1273 50  0000 C CNN
 F 2 "" H 6150 1100 50  0001 C CNN
@@
 	6150 1100 6150 1150
 $Comp
-L power:+3.3V #PWR?
+L power:+3.3V #PWR04
 U 1 1 602A8A27
 P 5100 3100
-F 0 "#PWR?" H 5100 2950 50  0001 C CNN
+F 0 "#PWR04" H 5100 2950 50  0001 C CNN
 F 1 "+3.3V" H 5115 3273 50  0000 C CNN
 F 2 "" H 5100 3100 50  0001 C CNN
@@
 	5100 3700 4900 3700
 $Comp
-L Device:L L?
+L Device:L L1
 U 1 1 602A9465
 P 6350 1000
-F 0 "L?" H 6403 1046 50  0000 L CNN
+F 0 "L1" H 6403 1046 50  0000 L CNN
 F 1 "L" H 6403 955 50  0000 L CNN
 F 2 "" H 6350 1000 50  0001 C CNN
@@
 	5950 850  5950 1150
 $Comp
-L Device:C C?
+L Device:C C4
 U 1 1 602ABE20
 P 4650 1550
-F 0 "C?" H 4765 1596 50  0000 L CNN
+F 0 "C4" H 4765 1596 50  0000 L CNN
 F 1 "C" H 4765 1505 50  0000 L CNN
 F 2 "" H 4688 1400 50  0001 C CNN
@@
 $EndComp
 $Comp
-L Device:C C?
+L Device:C C3
 U 1 1 602AC4D9
 P 4300 1550
-F 0 "C?" H 4415 1596 50  0000 L CNN
+F 0 "C3" H 4415 1596 50  0000 L CNN
 F 1 "C" H 4415 1505 50  0000 L CNN
 F 2 "" H 4338 1400 50  0001 C CNN
@@
 $EndComp
 $Comp
-L Device:C C?
+L Device:C C2
 U 1 1 602AC767
 P 3950 1550
-F 0 "C?" H 4065 1596 50  0000 L CNN
+F 0 "C2" H 4065 1596 50  0000 L CNN
 F 1 "C" H 4065 1505 50  0000 L CNN
 F 2 "" H 3988 1400 50  0001 C CNN
@@
 $EndComp
 $Comp
-L Device:C C?
+L Device:C C1
 U 1 1 602ACA9D
 P 3650 1550
-F 0 "C?" H 3765 1596 50  0000 L CNN
+F 0 "C1" H 3765 1596 50  0000 L CNN
 F 1 "C" H 3765 1505 50  0000 L CNN
 F 2 "" H 3688 1400 50  0001 C CNN
@@
 $EndComp
 $Comp
-L power:GND #PWR?
+L power:GND #PWR02
 U 1 1 602ACDD8
 P 4150 2050
-F 0 "#PWR?" H 4150 1800 50  0001 C CNN
+F 0 "#PWR02" H 4150 1800 50  0001 C CNN
 F 1 "GND" H 4155 1877 50  0000 C CNN
 F 2 "" H 4150 2050 50  0001 C CNN
@@
 	5650 850  5650 1300
 $Comp
-L Connector:Conn_01x02_Male J?
+L Connector:Conn_01x02_Male J5
 U 1 1 602B08AA
 P 7800 2200
-F 0 "J?" H 7772 2174 50  0000 R CNN
+F 0 "J5" H 7772 2174 50  0000 R CNN
 F 1 "Conn_01x02_Male" H 7772 2083 50  0000 R CNN
 F 2 "" H 7800 2200 50  0001 C CNN
@@
 	7600 2300 7050 2300
 $Comp
-L Connector:Conn_01x05_Male J?
+L Connector:Conn_01x05_Male J2
 U 1 1 602B2D83
 P 4700 550
-F 0 "J?" V 4762 794 50  0000 L CNN
+F 0 "J2" V 4762 794 50  0000 L CNN
 F 1 "Conn_01x05_Male" V 4853 794 50  0000 L CNN
 F 2 "" H 4700 550 50  0001 C CNN
@@
 	6150 1150 6150 1300
 $Comp
-L Connector:Conn_01x07_Male J?
+L Connector:Conn_01x07_Male J4
 U 1 1 602B70CA
 P 7800 1800
-F 0 "J?" H 7772 1824 50  0000 R CNN
+F 0 "J4" H 7772 1824 50  0000 R CNN
 F 1 "Conn_01x07_Male" H 7772 1733 50  0000 R CNN
 F 2 "" H 7800 1800 50  0001 C CNN
@@
 	7600 2100 7050 2100
 $Comp
-L Connector:Conn_01x07_Male J?
+L Connector:Conn_01x07_Male J6
 U 1 1 602BEFED
 P 7800 2700
-F 0 "J?" H 7772 2724 50  0000 R CNN
+F 0 "J6" H 7772 2724 50  0000 R CNN
 F 1 "Conn_01x07_Male" H 7772 2633 50  0000 R CNN
 F 2 "" H 7800 2700 50  0001 C CNN
@@
 	7600 3000 7050 3000
 $Comp
-L Connector:Conn_01x07_Male J?
+L Connector:Conn_01x07_Male J7
 U 1 1 602C721D
 P 7800 3400
-F 0 "J?" H 7772 3424 50  0000 R CNN
+F 0 "J7" H 7772 3424 50  0000 R CNN
 F 1 "Conn_01x07_Male" H 7772 3333 50  0000 R CNN
 F 2 "" H 7800 3400 50  0001 C CNN
@@
 	7600 3700 7050 3700
 $Comp
-L Connector:Conn_01x07_Male J?
+L Connector:Conn_01x07_Male J8
 U 1 1 602D1251
 P 7800 4100
-F 0 "J?" H 7772 4124 50  0000 R CNN
+F 0 "J8" H 7772 4124 50  0000 R CNN
 F 1 "Conn_01x07_Male" H 7772 4033 50  0000 R CNN
 F 2 "" H 7800 4100 50  0001 C CNN
@@
 	7450 4500 6150 4500
 $Comp
-L Connector:Conn_01x05_Male J?
+L Connector:Conn_01x05_Male J1
 U 1 1 602DCC1A
 P 4000 2650
-F 0 "J?" V 4062 2894 50  0000 L CNN
+F 0 "J1" V 4062 2894 50  0000 L CNN
 F 1 "Conn_01x05_Male" V 4153 2894 50  0000 L CNN
 F 2 "" H 4000 2650 50  0001 C CNN
@@
 $EndComp
 $Comp
-L power:GND #PWR?
+L power:GND #PWR01
 U 1 1 602DF078
 P 3800 3100
-F 0 "#PWR?" H 3800 2850 50  0001 C CNN
+F 0 "#PWR01" H 3800 2850 50  0001 C CNN
 F 1 "GND" H 3805 2927 50  0000 C CNN
 F 2 "" H 3800 3100 50  0001 C CNN
@@
 $EndComp
 $Comp
-L power:+3.3V #PWR?
+L power:+3.3V #PWR03
 U 1 1 602DF960
 P 4400 3200
-F 0 "#PWR?" H 4400 3050 50  0001 C CNN
+F 0 "#PWR03" H 4400 3050 50  0001 C CNN
 F 1 "+3.3V" H 4415 3373 50  0000 C CNN
 F 2 "" H 4400 3200 50  0001 C CNN
@@
 Text Label 9750 2100 0    50   ~ 0
 SDA
+Text GLabel 10150 2200 2    50   Input ~ 0
+CCS811_nINT
+Text GLabel 10150 2300 2    50   Input ~ 0
+CCS811_nRESET
+Text GLabel 10150 2400 2    50   Input ~ 0
+CCS811_nWAKE
+Text Label 7250 2400 0    50   ~ 0
+nINT
+Text Label 7250 2500 0    50   ~ 0
+nRST
+Text Label 7250 2600 0    50   ~ 0
+nWAKE
+Wire Wire Line
+	10150 2200 9750 2200
+Wire Wire Line
+	10150 2300 9750 2300
+Wire Wire Line
+	10150 2400 9750 2400
+Text Label 9750 2200 0    50   ~ 0
+nINT
+Text Label 9750 2300 0    50   ~ 0
+nRST
+Text Label 9750 2400 0    50   ~ 0
+nWAKE
+$Comp
+L Connector:Conn_01x08_Male J?
+U 1 1 60323D13
+P 1950 5500
+F 0 "J?" H 2058 5981 50  0000 C CNN
+F 1 "LCD" H 2058 5890 50  0000 C CNN
+F 2 "" H 1950 5500 50  0001 C CNN
+F 3 "~" H 1950 5500 50  0001 C CNN
+	1    1950 5500
+	1    0    0    -1
+$EndComp
+Wire Wire Line
+	2150 5300 2800 5300
+Wire Wire Line
+	2150 5400 2950 5400
+Wire Wire Line
+	2150 5500 2950 5500
+Wire Wire Line
+	2150 5600 2950 5600
+Wire Wire Line
+	2150 5700 2950 5700
+Wire Wire Line
+	2150 5800 2950 5800
+$Comp
+L power:+3.3V #PWR?
+U 1 1 6033BA4B
+P 2800 5000
+F 0 "#PWR?" H 2800 4850 50  0001 C CNN
+F 1 "+3.3V" H 2815 5173 50  0000 C CNN
+F 2 "" H 2800 5000 50  0001 C CNN
+F 3 "" H 2800 5000 50  0001 C CNN
+	1    2800 5000
+	1    0    0    -1
+$EndComp
+Wire Wire Line
+	2150 5900 2800 5900
+Wire Wire Line
+	2800 5000 2800 5100
+Connection ~ 2800 5300
+Wire Wire Line
+	2800 5300 2950 5300
+$Comp
+L power:GND #PWR?
+U 1 1 6034B03A
+P 2250 6050
+F 0 "#PWR?" H 2250 5800 50  0001 C CNN
+F 1 "GND" H 2255 5877 50  0000 C CNN
+F 2 "" H 2250 6050 50  0001 C CNN
+F 3 "" H 2250 6050 50  0001 C CNN
+	1    2250 6050
+	1    0    0    -1
+$EndComp
+Wire Wire Line
+	2250 6050 2250 5200
+Wire Wire Line
+	2150 5200 2250 5200
+Connection ~ 2250 5200
+Wire Wire Line
+	2250 5200 2950 5200
+Wire Wire Line
+	2800 5900 2800 6050
+Wire Wire Line
+	2800 6050 2350 6050
+Wire Wire Line
+	2350 6050 2350 5100
+Wire Wire Line
+	2350 5100 2800 5100
+Connection ~ 2800 5900
+Wire Wire Line
+	2800 5900 2950 5900
+Connection ~ 2800 5100
+Wire Wire Line
+	2800 5100 2800 5300
+Text Label 2950 5800 2    50   ~ 0
+dis_CS
+Text Label 2950 5700 2    50   ~ 0
+dis_RS
+Text Label 2950 5600 2    50   ~ 0
+dis_RES
+Text Label 2950 5500 2    50   ~ 0
+dis_SDA
+Text Label 2950 5400 2    50   ~ 0
+dis_SCK
+Text Label 7250 2700 0    50   ~ 0
+dis_SCK
+Text Label 7250 2800 0    50   ~ 0
+dis_SDA
+Text Label 7250 2900 0    50   ~ 0
+dis_RES
+Text Label 7250 3000 0    50   ~ 0
+dis_RS
+Text Label 7250 3100 0    50   ~ 0
+dis_CS
 $EndSCHEMATC
